File: amiga-500-usb-kb-stamp/amiga-500-usb-kb-stamp.kicad_pcb (KiCad board)
At the start: 2 copper layers, 48.8 x 43.9 mm, 18 parts, among them IC1 TXS0104ED, J1 USB3075-30-A, J2 USB_HEADER, J3 Type A, J4 Type B, J5 I2C, J6 DEBUG, J7 Power LED, J8 Floppy LED, J9 USB_BOOT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

Commit message: Add files via upload
Parts:
- R1: value 4.7k -> 10k
Connections:
- IC1 pad 6: Net-(IC1-Pad6) -> (no net)
- IC1 pad 7: Net-(IC1-Pad7) -> GND
- IC1 pad 9: Net-(IC1-Pad9) -> (no net)
- J1 pad 4: Net-(J1-Pad4) -> (no net)
- J3 pad 5: Net-(J3-Pad5) -> (no net)
- J4 pad 5: Net-(J4-Pad5) -> (no net)
Other:
- board text added: "rev 2"
- board text added: "wiretap 2024"
- board text removed: "rev 1"
- board text removed: "wiretap 2022"
