File: amiga-500-usb-kb-stamp/amiga-500-usb-kb-stamp.sch (KiCad schematic (older format))
At the start: 17 parts, among them IC1 TXS0104ED, J1 USB3075-30-A, J2 USB_HEADER, J3 Type A, J4 Type B, J5 I2C, J6 DEBUG, J7 Power LED, J8 Floppy LED, J9 USB_BOOT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

Commit message: Add files via upload
Connections:
- net GND: now also IC1.7 (GND)
Changed lines of the file:
@@
 Sheet 1 1
 Title "A500 RP2040 Stamp Keyboard Adapter"
-Date "2022-08-02"
-Rev "1"
+Date "2024-01-16"
+Rev "2"
 Comp "wiretap"
 Comment1 ""
@@
 KB_CLK_RAW
 Wire Wire Line
-	3250 4050 5550 4050
+	3250 4050 3800 4050
 Wire Wire Line
 	5550 3200 5250 3200
@@
 	900  2250 900  1750
 Connection ~ 900  1750
+Wire Wire Line
+	3800 3800 3800 4050
+Connection ~ 3800 4050
+Wire Wire Line
+	3800 4050 5550 4050
 $EndSCHEMATC
